File: Picobreadboad_PCB.kicad_pcb (KiCad board)
At the start: 2 copper layers, 104 x 66 mm, 10 parts, among them J1 Conn_02x20_Odd_Even, J14 Conn_02x20_Odd_Even, J16 Conn_02x20_Odd_Even, J2 Conn_02x20_Odd_Even, J3 Conn_02x20_Odd_Even, J4 Conn_02x20_Odd_Even

Commit message: kicadfile
Parts:
- added G***: LOGO, logo:logo_dongdo_korean_small3, B.Cu at (132.8, 92.9)
- added G***: LOGO, logo:logo_dongdo_small3, B.Cu at (128.2, 73.6)
Connections:
- J1 pad 15: Net-(J1-Pin_15) -> GND
- J1 pad 16: Net-(J1-Pin_15) -> GND
- J1 pad 25: Net-(J1-Pin_25) -> GND
- J1 pad 26: Net-(J1-Pin_25) -> GND
- J1 pad 35: Net-(J1-Pin_35) -> GND
- J1 pad 36: Net-(J1-Pin_35) -> GND
- J1 pad 5: Net-(J1-Pin_5) -> GND
- J1 pad 6: Net-(J1-Pin_5) -> GND
- J14 pad 15: Net-(J14-Pin_15) -> GND
- J14 pad 16: Net-(J14-Pin_15) -> GND
- J14 pad 25: Net-(J14-Pin_25) -> GND
- J14 pad 26: Net-(J14-Pin_25) -> GND
- J14 pad 35: Net-(J14-Pin_35) -> GND
- J14 pad 36: Net-(J14-Pin_35) -> GND
- J14 pad 5: Net-(J14-Pin_5) -> GND
- J14 pad 6: Net-(J14-Pin_5) -> GND
- J16 pad 15: Net-(J1-Pin_15) -> GND
- J16 pad 16: Net-(J1-Pin_15) -> GND
- J16 pad 25: Net-(J1-Pin_25) -> GND
- J16 pad 26: Net-(J1-Pin_25) -> GND
- J16 pad 35: Net-(J1-Pin_35) -> GND
- J16 pad 36: Net-(J1-Pin_35) -> GND
- J16 pad 5: Net-(J1-Pin_5) -> GND
- J16 pad 6: Net-(J1-Pin_5) -> GND
- J2 pad 15: Net-(J14-Pin_15) -> GND
- J2 pad 16: Net-(J14-Pin_15) -> GND
- J2 pad 25: Net-(J14-Pin_25) -> GND
- J2 pad 26: Net-(J14-Pin_25) -> GND
- J2 pad 35: Net-(J14-Pin_35) -> GND
- J2 pad 36: Net-(J14-Pin_35) -> GND
- J2 pad 5: Net-(J14-Pin_5) -> GND
- J2 pad 6: Net-(J14-Pin_5) -> GND
- J3 pad 15: Net-(J1-Pin_15) -> GND
- J3 pad 16: Net-(J1-Pin_15) -> GND
- J3 pad 25: Net-(J1-Pin_25) -> GND
- J3 pad 26: Net-(J1-Pin_25) -> GND
- J3 pad 35: Net-(J1-Pin_35) -> GND
- J3 pad 36: Net-(J1-Pin_35) -> GND
- J3 pad 5: Net-(J1-Pin_5) -> GND
- J3 pad 6: Net-(J1-Pin_5) -> GND
- J4 pad 15: Net-(J14-Pin_15) -> GND
- J4 pad 16: Net-(J14-Pin_15) -> GND
- J4 pad 25: Net-(J14-Pin_25) -> GND
- J4 pad 26: Net-(J14-Pin_25) -> GND
- J4 pad 35: Net-(J14-Pin_35) -> GND
- J4 pad 36: Net-(J14-Pin_35) -> GND
- J4 pad 5: Net-(J14-Pin_5) -> GND
- J4 pad 6: Net-(J14-Pin_5) -> GND
Routing:
- net GND: track 206.0 -> 518.0 mm
- net Net-(J14-Pin_25): track 33.0 -> 0.00 mm
- net Net-(J14-Pin_35): track 33.0 -> 0.00 mm
- net Net-(J14-Pin_5): track 33.0 -> 0.00 mm
- net Net-(J14-Pin_15): track 33.0 -> 0.00 mm
- net Net-(J1-Pin_5): track 32.6 -> 0.00 mm
- net Net-(J1-Pin_35): track 32.6 -> 0.00 mm
- net Net-(J1-Pin_25): track 32.6 -> 0.00 mm
- net Net-(J1-Pin_15): track 32.6 -> 0.00 mm
