File: Picobreadboad_PCB.kicad_sch (KiCad schematic)
At the start: 11 parts, among them IC1 RASPBERRY_PI_PICO_W, J1 Conn_02x20_Odd_Even, J14 Conn_02x20_Odd_Even, J16 Conn_02x20_Odd_Even, J2 Conn_02x20_Odd_Even, J3 Conn_02x20_Odd_Even, J4 Conn_02x20_Odd_Even

Commit message: kicadfile
Connections:
- net GND: now also IC1.13 (GND_3), IC1.18 (GND_4), IC1.23 (GND_5), IC1.28 (GND_6), IC1.3 (GND_1), IC1.33 (GND/AGND), IC1.38 (GND_7), IC1.8 (GND_2), J1.15 (Pin_15), J1.16 (Pin_16), J1.25 (Pin_25), J1.26 (Pin_26)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
